Commit message: Wire real ground-truth wheel contact telemetry into the ledge-test path
Track B.1: give the balance/landing path real per-wheel contact sensing,
observational only. Previously Gazebo contact sensing existed only for the
jump_model path (run_jump.sh); the plain balance/ledge-test path
(run_sim.sh, clean_ledge_smoke.py) relied entirely on the pose+IMU
floor_contact heuristic with no real ground truth available at all.

Added a new, independent measure_contacts:=true launch arg (decoupled from
jump_model so it doesn't also swap in BoundedGazeboSystem/lower actuator
limits) that enables the wheel contact sensors on ledge_test.sdf (now loads
gz-sim-contact-system). BalanceControllerNode already always subscribes to
left/right wheel contacts regardless of jump.enabled, so no C++ changes were
needed - only the Gazebo-side wiring was missing.

Along the way found libtap_contact_snapshot.so intermittently fails to load
in this environment (libsystemd version mismatch, unrelated to its own
code), so the bridge now reads the sensor's own _raw topic directly instead
of depending on that plugin. This drops the documented "empty sample
confirms airborne" guarantee for consumers of /left_wheel_contacts -
documented the caveat in CONTRACT.md.

Deliberately does NOT feed floor_contact or any control decision: three
earlier attempts in docs/LEDGE_DRIVEOFF_LIMIT.md to make floor_contact react
to a better/faster sensor all measurably hurt or tied at best, so doing that
again with yet another sensor would likely repeat the same failed
experiment. This is pure telemetry, verified end-to-end with a real
drive-off-the-ledge trial (9876 samples, 8390 with real contact=1, 5303
fresh) - a foundation for a future kinematics-estimated Fz/friction-cone
term, not a change to current production behavior. Confirmed zero effect on
the default (measure_contacts left false) path via sim_smoke.py and a fresh
clean_ledge_smoke.py --skip-enabled batch.

Co-Authored-By: Claude Sonnet 5 <noreply@anthropic.com>

File: src/tap_robot_description/description/cad_robot/robot.urdf.xacro (robot description, xacro)
@@ -6,6 +6,11 @@
   <xacro:arg name="jump_leg_speed" default="12.566370614359172"/>
   <xacro:arg name="jump_leg_velocity_damping" default="0.0"/>
+  <!-- Wheel contact sensors only, decoupled from jump_model's actuator-bound
+       swap (BoundedGazeboSystem, lower effort/velocity limits) below. Opt-in
+       and additive: leaves every non-jump default behavior unchanged. -->
+  <xacro:arg name="measure_contacts" default="false"/>
   <xacro:property name="jump_leg_speed" value="${float('$(arg jump_leg_speed)')}"/>
   <xacro:property name="jump_model" value="${'$(arg jump_model)' == 'true' and '$(arg simulation)' == 'true'}"/>
+  <xacro:property name="measure_contacts" value="${'$(arg measure_contacts)' == 'true' and '$(arg simulation)' == 'true'}"/>
   <xacro:property name="simulation" value="${'$(arg simulation)' == 'true'}"/>
   <xacro:property name="mesh_root" value="package://tap_robot_description/description/cad_robot/meshes"/>

File: src/tap_robot_description/description/cad_robot/simulation.urdf.xacro (robot description, xacro)
@@ -58,5 +58,5 @@
   <gazebo reference="cad_left_wheel_link"><mu1>1.0</mu1><mu2>1.0</mu2></gazebo>
   <gazebo reference="cad_right_wheel_link"><mu1>1.0</mu1><mu2>1.0</mu2></gazebo>
-  <xacro:if value="${jump_model}">
+  <xacro:if value="${jump_model or measure_contacts}">
     <gazebo>
       <plugin filename="$(find tap_sim)/../../lib/libtap_contact_snapshot.so" name="tap_sim::ContactSnapshot"/>
